File: Thunderbread.sch (EAGLE design)
At the start: 57 parts, among them K1 S102S02, Q1 TIP120, Q2 TIP120, T1 2N2222, U1 ARDUINO-MEGAFULL, X1 HD44780LCD-1602

Commit message: Diameter sensor & starve feeder rewired
Connections:
- removed net N$27: U$9.A4, U1.20(SDA)
- removed net N$30: U$9.A5, U1.21(SCL)
- new net DIAMETER_SENSOR_5V: U$9.+5V
- new net DIAMETER_SENSOR_GND: U$9.GND1
- new net DIAMETER_SENSOR_SIGNAL: U$9.A0
- new net DIR_BALANCE: U$8.D5
- new net ENABLE_BALANCE: U$8.D3
- new net OPTICAL_SLOT_BALANCE: U$8.D2
- new net SCL: U$8.A4, U$9.A4, U1.20(SDA)
- new net SDA: U$8.A5, U$9.A5, U1.21(SCL)
- new net STEP_BALANCE: U$8.D4
Other:
- note removed: "Diameter Sensor +5V"
- note removed: "Diameter Sensor GND"
- note removed: "Diameter Sensor Signal"
- note removed: "Dir (Balance)"
- note removed: "Enable (Balance)"
- note removed: "Optical Slot (Balance)"
- note removed: "SCL"
- note removed: "SDA"
- note removed: "Step (Balance)"
- moved on the sheet: #, *, 0, 1, 2, 3, 4, 5, 6, 7, 8, 9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
